Commit message: working on description/gazeebo

File: urdf/raptor.urdf.xacro (robot description, xacro)
@@ -1,8 +1,10 @@
 <?xml version="1.0"?>
-	<robot name="raptor">
+	<robot name="raptor" xmlns:xacro="http://www.ros.org/wiki/xacro">
+	<xacro:include filename="$(find raptor_robot)/urdf/include/material.xacro"/>
+	<xacro:include filename="$(find raptor_robot)/urdf/include/gazebo.xacro"/>
   		<link name="base_link">
 		</link>
 		<link name="chassis_frame">
-			<visual>
+			<collision>
 			<geometry>
 				<box size="0.80 0.54 0.22"/>
@@ -12,13 +14,40 @@
 				<color rgba="1 0 0 1"/>
 			</material>
-			<!--
-			<material name="yellow">
-				<color rgba="0.8 0.8 0.0 1" />
-			</material>
-			<material name="white">
-				<color rgba="1 1 1 1"/>
-			</material>
-			-->
-			</visual>
+			</collision>
+			<visual>
+			<geometry>
+				<box size="0.80 0.54 0.22"/>
+			</geometry>
+			<origin rpy="0 0 0" xyz="0 0 0.10"/>
+			<material name="red">
+				<color rgba="1 0 0 1"/>
+			</material>
+			</visual>
+			<!-- caster -->
+			<collision name="caster_rear_collision">
+    			<origin rpy=" 0 0 0" xyz="-0.38 0 0.01"/>
+    			<geometry>
+      				<sphere radius="0.11"/>
+    			</geometry>
+    			<surface>
+      				<friction>
+        				<ode>
+          					<mu>0</mu>
+          					<mu2>0</mu2>
+          					<slip1>1.0</slip1>
+          					<slip2>1.0</slip2>
+        				</ode>
+      				</friction>
+    			</surface>
+  			</collision>
+  			<visual name="caster_rear_visual">
+    			<origin rpy=" 0 0 0" xyz="-0.38 0 0.01"/>
+    			<geometry>
+      				<sphere radius="0.11"/>
+    			</geometry>
+				<material name="black">
+					<color rgba="0.0 0.0 0.0 1.0"/>
+				</material>
+  			</visual>
 		</link>
 		<joint name="base_to_chassis_frame" type="fixed">
@@ -134,5 +163,5 @@
 			</visual>
   		</link>
-		<joint name="base_to_lwheel" type="fixed">
+		<joint name="base_to_lwheel" type="continuous">
 			<parent link="base_link"/>
 			<child link="lwheel"/>
@@ -150,5 +179,5 @@
 			</visual>
 		</link>
-		<joint name="base_to_rwheel" type="fixed">
+		<joint name="base_to_rwheel" type="continuous">
 			<parent link="base_link"/>
 			<child link="rwheel"/>
@@ -268,41 +297,3 @@
 			<axis xyz="0 0 0"/>
 		</joint>
-		<gazebo>
-			<plugin name="differential_drive_controller" filename="libgazebo_ros_diff_drive.so">
-				<!-- Plugin update rate in Hz
-				<updateRate>${update_rate}</updateRate>
-				-->
-				<updateRate>10</updateRate>
-				<!-- Name of left joint, defaults to `left_joint` -->
-				<leftJoint>base_to_lwheel</leftJoint>
-				<!-- Name of right joint, defaults to `right_joint` -->
-				<rightJoint>base_to_rwheel</rightJoint>
-				<!-- The distance from the center of one wheel to the other, in meters, defaults to 0.34 m -->
-				<wheelSeparation>0.45</wheelSeparation>
-				<!-- Diameter of the wheels, in meters, defaults to 0.15 m -->
-				<wheelDiameter>0.285</wheelDiameter>
-				<!-- Wheel acceleration, in rad/s^2, defaults to 0.0 rad/s^2 -->
-				<wheelAcceleration>1.0</wheelAcceleration>
-				<!-- Maximum torque which the wheels can produce, in Nm, defaults to 5 Nm -->
-				<wheelTorque>20</wheelTorque>
-				<!-- Topic to receive geometry_msgs/Twist message commands, defaults to `cmd_vel` -->
-				<commandTopic>cmd_vel</commandTopic>
-				<!-- Topic to publish nav_msgs/Odometry messages, defaults to `odom` -->
-				<odometryTopic>odom</odometryTopic>
-				<!-- Odometry frame, defaults to `odom` -->
-				<odometryFrame>odom</odometryFrame>
-				<!-- Robot frame to calculate odometry from, defaults to `base_footprint` -->
-				<robotBaseFrame>base_footprint</robotBaseFrame>
-				<!-- Odometry source, 0 for ENCODER, 1 for WORLD, defaults to WORLD -->
-				<odometrySource>1</odometrySource>
-				<!-- Set to true to publish transforms for the wheel links, defaults to false -->
-				<publishWheelTF>true</publishWheelTF>
-				<!-- Set to true to publish transforms for the odometry, defaults to true -->
-				<publishOdom>true</publishOdom>
-				<!-- Set to true to publish sensor_msgs/JointState on /joint_states for the wheel joints, defaults to false -->
-				<publishWheelJointState>true</publishWheelJointState>
-				<!-- Set to true to swap right and left wheels, defaults to true -->
-				<legacyMode>false</legacyMode>
-			</plugin>
-		</gazebo>
 	</robot>

Commit message: got gazebo launch spawning robot, needs iniertial tags edited

File: urdf/raptor.urdf.xacro (robot description, xacro)
@@ -6,4 +6,9 @@
 		</link>
 		<link name="chassis_frame">
+		<inertial>
+      		<origin xyz="0 0 0" rpy="0 0 0"/>
+      		<mass value="1.0" />
+      		<inertia ixx="0.0741666666667" ixy="0.0" ixz="0.0" iyy="0.0585416666667" iyz="0.0" izz="0.0260416666667"/>
+		</inertial>
 			<collision>
 			<geometry>
@@ -57,4 +62,9 @@
 		</joint>
 		<link name="pvc_up_left">
+			<inertial>
+      			<origin xyz="0 0 0" rpy="0 0 0"/>
+      			<mass value="1.0" />
+      			<inertia ixx="0.0741666666667" ixy="0.0" ixz="0.0" iyy="0.0585416666667" iyz="0.0" izz="0.0260416666667"/>
+			</inertial>
 			<visual>
 			<geometry>
@@ -73,4 +83,9 @@
 		</joint>
 		<link name="pvc_up_right">
+			<inertial>
+      			<origin xyz="0 0 0" rpy="0 0 0"/>
+      			<mass value="1.0" />
+      			<inertia ixx="0.0741666666667" ixy="0.0" ixz="0.0" iyy="0.0585416666667" iyz="0.0" izz="0.0260416666667"/>
+			</inertial>
 			<visual>
 			<geometry>
@@ -89,4 +104,9 @@
 		</joint>
 		<link name="pvc_horizontal">
+			<inertial>
+      			<origin xyz="0 0 0" rpy="0 0 0"/>
+      			<mass value="1.0" />
+      			<inertia ixx="0.0741666666667" ixy="0.0" ixz="0.0" iyy="0.0585416666667" iyz="0.0" izz="0.0260416666667"/>
+			</inertial>
 			<visual>
 			<geometry>
@@ -105,4 +125,9 @@
 		</joint>
 		<link name="pvc_45_left">
+			<inertial>
+      			<origin xyz="0 0 0" rpy="0 0 0"/>
+      			<mass value="1.0" />
+      			<inertia ixx="0.0741666666667" ixy="0.0" ixz="0.0" iyy="0.0585416666667" iyz="0.0" izz="0.0260416666667"/>
+			</inertial>
 			<visual>
 			<geometry>
@@ -121,4 +146,9 @@
 		</joint>
 		<link name="pvc_45_right">
+			<inertial>
+      			<origin xyz="0 0 0" rpy="0 0 0"/>
+      			<mass value="1.0" />
+      			<inertia ixx="0.0741666666667" ixy="0.0" ixz="0.0" iyy="0.0585416666667" iyz="0.0" izz="0.0260416666667"/>
+			</inertial>
 			<visual>
 			<geometry>
@@ -137,4 +167,9 @@
 		</joint>
 		<link name="bucket">
+			<inertial>
+      			<origin xyz="0 0 0" rpy="0 0 0"/>
+      			<mass value="1.0" />
+      			<inertia ixx="0.0741666666667" ixy="0.0" ixz="0.0" iyy="0.0585416666667" iyz="0.0" izz="0.0260416666667"/>
+			</inertial>
 			<visual>
 			<geometry>
@@ -153,4 +188,15 @@
 		</joint>
 		<link name="lwheel">
+			<inertial>
+      			<origin xyz="0 0 0" rpy="0 0 0"/>
+      			<mass value="1.0" />
+      			<inertia ixx="0.0741666666667" ixy="0.0" ixz="0.0" iyy="0.0585416666667" iyz="0.0" izz="0.0260416666667"/>
+			</inertial>
+			<collision name="lwheel_collision">
+    			<origin rpy=" 0 0 0" xyz="0 0 0"/>
+    			<geometry>
+      				<cylinder length="0.07" radius="0.14"/>
+    			</geometry>
+  			</collision>
 			<visual>
 			<geometry>
@@ -169,4 +215,15 @@
 		</joint>
 		<link name="rwheel">
+			<inertial>
+      			<origin xyz="0 0 0" rpy="0 0 0"/>
+      			<mass value="1.0" />
+      			<inertia ixx="0.0741666666667" ixy="0.0" ixz="0.0" iyy="0.0585416666667" iyz="0.0" izz="0.0260416666667"/>
+			</inertial>
+			<collision name="rwheel_collision">
+    			<origin rpy=" 0 0 0" xyz="0 0 0"/>
+    			<geometry>
+      				<cylinder length="0.07" radius="0.14"/>
+    			</geometry>
+  			</collision>
 			<visual>
 			<geometry>
@@ -185,4 +242,9 @@
 		</joint>
 		<link name="front_laser">
+			<inertial>
+      			<origin xyz="0 0 0" rpy="0 0 0"/>
+      			<mass value="1.0" />
+      			<inertia ixx="0.0741666666667" ixy="0.0" ixz="0.0" iyy="0.0585416666667" iyz="0.0" izz="0.0260416666667"/>
+			</inertial>
 			<visual>
 			<geometry>
@@ -211,4 +273,9 @@
 		</joint>
 		<link name="scan_multi">
+			<inertial>
+      			<origin xyz="0 0 0" rpy="0 0 0"/>
+      			<mass value="1.0" />
+      			<inertia ixx="0.0741666666667" ixy="0.0" ixz="0.0" iyy="0.0585416666667" iyz="0.0" izz="0.0260416666667"/>
+			</inertial>
 			<visual>
 			<geometry>
@@ -237,4 +304,9 @@
 		</joint>
 		<link name="rear_laser">
+			<inertial>
+      			<origin xyz="0 0 0" rpy="0 0 0"/>
+      			<mass value="1.0" />
+      			<inertia ixx="0.0741666666667" ixy="0.0" ixz="0.0" iyy="0.0585416666667" iyz="0.0" izz="0.0260416666667"/>
+			</inertial>
 			<visual>
 			<geometry>
@@ -264,4 +336,9 @@
 		<!-- Camera -->
 		<link name="camera_link">
+			<inertial>
+      			<origin xyz="0 0 0" rpy="0 0 0"/>
+      			<mass value="1.0" />
+      			<inertia ixx="0.0741666666667" ixy="0.0" ixz="0.0" iyy="0.0585416666667" iyz="0.0" izz="0.0260416666667"/>
+			</inertial>
 			<!-- <inertial>
 				<mass value="${camera_mass}"/>

Commit message: fixing stuff on robot hardware

File: urdf/raptor.urdf.xacro (robot description, xacro)
@@ -279,5 +279,5 @@
 			<axis xyz="0.0 0.0 1.0"/>
 		</joint>
-		<link name="front_laser">
+		<link name="laser">
 			<inertial>
       			<origin xyz="0 0 0" rpy="0 0 0"/>
@@ -303,5 +303,5 @@
 		<joint name="base_link_to_front_laser" type="fixed">
 			<parent link="base_link"/>
-			<child link="front_laser"/>
+			<child link="laser"/>
 			<!--
 			<origin xyz="0.163 0 0.3" rpy="0.0 0.0 3.141592"/>

Commit message: adding mpu6050 to help odometery

File: urdf/raptor.urdf.xacro (robot description, xacro)
@@ -61,4 +61,20 @@
 			<origin xyz="0 0 0.10" rpy="0 0 0"/>
 		</joint>
+		<joint name="imu_joint" type="fixed">
+			<origin xyz="0 0 0" rpy="0 0 0" />
+			<parent link="base_link" />
+			<child link="imu_link" />
+		</joint>
+		<link name="imu_link">
+		<!--
+		<visual>
+		<origin rpy="0 0 1.5708" xyz="0 0 0"/>
+		<geometry>
+			<mesh filename="package://mpu_6050_driver/mesh/FUGMJ38JX8T7E5A.stl" scale="0.01 0.01 0.01"/>
+		</geometry>
+		<material name="white"/>
+		</visual>
+		-->
+		</link>
 		<link name="pvc_up_left">
 			<inertial>

Commit message: mounted mpu6050

File: urdf/raptor.urdf.xacro (robot description, xacro)
@@ -62,5 +62,5 @@
 		</joint>
 		<joint name="imu_joint" type="fixed">
-			<origin xyz="0 0 0" rpy="0 0 0" />
+			<origin xyz="0.35 0.02 0.39" rpy="0 0 0" />
 			<parent link="base_link" />
 			<child link="imu_link" />
