Commit message: 3d mapping works, need to test it :D

File: urdf/include/_d435i.urdf.xacro (robot description, xacro)
@@ -7,9 +7,8 @@
 -->
 <robot name="sensor_d435i" xmlns:xacro="http://ros.org/wiki/xacro">
-  <xacro:include filename="$(find realsense2_description)/urdf/_d435.urdf.xacro"/>
+  <xacro:include filename="$(find raptor_robot)/urdf/include/_d435.urdf.xacro"/>
   <xacro:include filename="$(find realsense2_description)/urdf/_d435i_imu_modules.urdf.xacro"/>
-  <xacro:macro name="sensor_d435i" params="parent *origin name:=camera use_nominal_extrinsics:=false">
+  <xacro:macro name="sensor_d435i" params="parent name:=camera use_nominal_extrinsics:=false">
     <xacro:sensor_d435 parent="${parent}" name="${name}" use_nominal_extrinsics="${use_nominal_extrinsics}">
-      <xacro:insert_block name="origin" />
     </xacro:sensor_d435>
     <xacro:d435i_imu_modules name="${name}" use_nominal_extrinsics="${use_nominal_extrinsics}"/>

File: urdf/raptor.urdf.xacro (robot description, xacro)
@@ -3,4 +3,5 @@
 	<xacro:include filename="$(find raptor_robot)/urdf/include/material.xacro"/>
 	<xacro:include filename="$(find raptor_robot)/urdf/include/gazebo.xacro"/>
+	<xacro:include filename="$(find raptor_robot)/urdf/include/_d435i.urdf.xacro"/>
   		<link name="base_link">
 		</link>
@@ -388,5 +389,5 @@
 			<axis xyz="0 0 0"/>
 		</joint>
-		<!-- Camera -->
+		<!-- Camera
 		<link name="camera_link">
 			<inertial>
@@ -411,5 +412,6 @@
 			</collision>
 		</link>
-		<!-- Camera Joint -->
+-->
+		<!-- Camera Joint
 		<joint name="camera_joint" type="fixed">
 			<origin xyz="-0.16 0 0.93" rpy="0 0 0" />
@@ -418,3 +420,6 @@
 			<axis xyz="0 0 0"/>
 		</joint>
+-->
+		<xacro:sensor_d435i parent="base_link">
+		</xacro:sensor_d435i>
 	</robot>
