Commit message: edit description for gazebo use

File: urdf/include/gazebo.xacro (robot description, xacro)
@@ -36,6 +36,6 @@
           <samples>720</samples>
           <resolution>1</resolution>
-          <min_angle>-1.570796</min_angle>
-          <max_angle>1.570796</max_angle>
+          <min_angle>-3.14</min_angle>
+          <max_angle>3.14</max_angle>
         </horizontal>
       </scan>
@@ -57,4 +57,37 @@
   </sensor>
 </gazebo>
+<!--
+<gazebo reference="rear_laser">
+  <sensor type="ray" name="head_hokuyo_sensor">
+    <pose>0 0 0 0 0 0</pose>
+    <visualize>false</visualize>
+    <update_rate>20</update_rate>
+    <ray>
+      <scan>
+        <horizontal>
+          <samples>720</samples>
+          <resolution>1</resolution>
+          <min_angle>-3.14</min_angle>
+          <max_angle>3.14</max_angle>
+        </horizontal>
+      </scan>
+      <range>
+        <min>0.10</min>
+        <max>10.0</max>
+        <resolution>0.01</resolution>
+      </range>
+      <noise>
+        <type>gaussian</type>
+        <mean>0.0</mean>
+        <stddev>0.01</stddev>
+      </noise>
+    </ray>
+    <plugin name="gazebo_ros_head_hokuyo_controller2" filename="libgazebo_ros_laser.so">
+      <topicName>/rear_laser_scan</topicName>
+      <frameName>laser</frameName>
+    </plugin>
+  </sensor>
+</gazebo>
+-->
 <gazebo reference="chassis_frame">
   <visual name="caster_front_visual">

File: urdf/raptor.urdf.xacro (robot description, xacro)
@@ -76,4 +76,10 @@
 			</material>
 			</visual>
+			<collision>
+				<origin xyz="0 0 0" rpy="0 0 0"/>
+				<geometry>
+					<cylinder length="0.54" radius="0.014"/>
+				</geometry>
+			</collision>
 		</link>
 		<joint name="pvc_up_left_to_chassis_frame" type="fixed">
@@ -97,4 +103,10 @@
 			</material>
 			</visual>
+			<collision>
+				<origin xyz="0 0 0" rpy="0 0 0"/>
+				<geometry>
+					<cylinder length="0.54" radius="0.014"/>
+				</geometry>
+			</collision>
 		</link>
 		<joint name="pvc_up_right_to_chassis_frame" type="fixed">
@@ -118,4 +130,10 @@
 			</material>
 			</visual>
+			<collision>
+				<origin xyz="0 0 0" rpy="0 0 0"/>
+				<geometry>
+					<cylinder length="0.4" radius="0.014"/>
+				</geometry>
+			</collision>
 		</link>
 		<joint name="pvc_horizontal_to_chassis_frame" type="fixed">
@@ -139,4 +157,10 @@
 			</material>
 			</visual>
+			<collision>
+				<origin xyz="0 0 0" rpy="0 0 0"/>
+				<geometry>
+					<cylinder length="0.64" radius="0.014"/>
+				</geometry>
+			</collision>
 		</link>
 		<joint name="pvc_45_left_to_chassis_frame" type="fixed">
@@ -160,4 +184,10 @@
 			</material>
 			</visual>
+			<collision>
+				<origin xyz="0 0 0" rpy="0 0 0"/>
+				<geometry>
+					<cylinder length="0.64" radius="0.014"/>
+				</geometry>
+			</collision>
 		</link>
 		<joint name="pvc_45_right_to_chassis_frame" type="fixed">
@@ -181,4 +211,10 @@
       		</material>
 			</visual>
+			<collision>
+				<origin xyz="0 0 0" rpy="0 0 0"/>
+				<geometry>
+					<cylinder length="0.36" radius="0.15"/>
+				</geometry>
+			</collision>
 		</link>
 		<joint name="bucket_to_chassis_frame" type="fixed">
@@ -341,14 +377,4 @@
       			<inertia ixx="0.0741666666667" ixy="0.0" ixz="0.0" iyy="0.0585416666667" iyz="0.0" izz="0.0260416666667"/>
 			</inertial>
-			<!-- <inertial>
-				<mass value="${camera_mass}"/>
-				<origin xyz="0 0 0" rpy="0 0 0"/>
-				<inertia
-					ixx="1e-6" ixy="0.0" ixz="0.0"
-					iyy="1e-6" iyz="0.0"
-					izz="1e-6"
-				/>
-			</inertial>
-			-->
 			<visual>
 				<origin xyz="0 0 0" rpy="0 0 0"/>

Commit message: more sim stuff

File: urdf/include/gazebo.xacro (robot description, xacro)
@@ -29,5 +29,5 @@
   <sensor type="ray" name="head_hokuyo_sensor">
     <pose>0 0 0 0 0 0</pose>
-    <visualize>true</visualize>
+    <visualize>false</visualize>
     <update_rate>20</update_rate>
     <ray>
@@ -53,9 +53,8 @@
     <plugin name="gazebo_ros_head_hokuyo_controller" filename="libgazebo_ros_laser.so">
       <topicName>/scan</topicName>
-      <frameName>laser</frameName>
+      <frameName>front_laser</frameName>
     </plugin>
   </sensor>
 </gazebo>
-<!--
 <gazebo reference="rear_laser">
   <sensor type="ray" name="head_hokuyo_sensor">
@@ -85,9 +84,8 @@
     <plugin name="gazebo_ros_head_hokuyo_controller2" filename="libgazebo_ros_laser.so">
       <topicName>/rear_laser_scan</topicName>
-      <frameName>laser</frameName>
+      <frameName>rear_laser</frameName>
     </plugin>
   </sensor>
 </gazebo>
--->
 <gazebo reference="chassis_frame">
   <visual name="caster_front_visual">

File: urdf/raptor.urdf.xacro (robot description, xacro)
@@ -249,4 +249,5 @@
 			<child link="lwheel"/>
 			<origin xyz="0.13 0.21 0.14" rpy="1.5708 0 0"/>
+			<axis xyz="0.0 0.0 -1.0"/>
 		</joint>
 		<link name="rwheel">
@@ -276,4 +277,5 @@
 			<child link="rwheel"/>
 			<origin xyz="0.13 -0.21 0.14" rpy="-1.5708 0 0"/>
+			<axis xyz="0.0 0.0 1.0"/>
 		</joint>
 		<link name="front_laser">

Commit message: Update gazebo.xacro

File: urdf/include/gazebo.xacro (robot description, xacro)
@@ -95,5 +95,5 @@
       <script>
         <uri>file://media/materials/scripts/gazebo.material</uri>
-        <name>Gazebo/Orange</name>
+        <name>Gazebo/Red</name>
       </script>
     </material>
@@ -101,8 +101,8 @@
 </gazebo>
 <gazebo reference="lwheel">
-  <material>Gazebo/Blue</material>
+  <material>Gazebo/Black</material>
 </gazebo>
 <gazebo reference="rwheel">
-  <material>Gazebo/Blue</material>
+  <material>Gazebo/Black</material>
 </gazebo>
 </robot>

Commit message: Update gazebo.xacro

File: urdf/include/gazebo.xacro (robot description, xacro)
@@ -106,3 +106,8 @@
   <material>Gazebo/Black</material>
 </gazebo>
+<gazebo reference="caster_wheel">
+  <material>Gazebo/Black</material>
+  <mu1>0.001</mu1>
+  <mu2>0.001</mu2>
+</gazebo>
 </robot>

Commit message: Update gazebo.xacro

File: urdf/include/gazebo.xacro (robot description, xacro)
@@ -9,5 +9,5 @@
     <leftJoint>base_to_lwheel</leftJoint>
     <rightJoint>base_to_rwheel</rightJoint>
-    <wheelSeparation>0.45</wheelSeparation>
+    <wheelSeparation>0.34</wheelSeparation>
     <wheelDiameter>0.2</wheelDiameter>
     <torque>0.1</torque>
@@ -30,5 +30,5 @@
     <pose>0 0 0 0 0 0</pose>
     <visualize>false</visualize>
-    <update_rate>20</update_rate>
+    <update_rate>10</update_rate>
     <ray>
       <scan>
@@ -106,8 +106,11 @@
   <material>Gazebo/Black</material>
 </gazebo>
-<gazebo reference="caster_wheel">
+<gazebo reference="caster_rear_collision">
   <material>Gazebo/Black</material>
   <mu1>0.001</mu1>
   <mu2>0.001</mu2>
 </gazebo>
+<gazebo reference="bucket">
+  <material>Gazebo/Blue</material>
+</gazebo>
 </robot>

Commit message: Update gazebo.xacro

File: urdf/include/gazebo.xacro (robot description, xacro)
@@ -114,3 +114,18 @@
   <material>Gazebo/Blue</material>
 </gazebo>
+<gazebo reference="pvc_horizontal">
+  <material>Gazebo/Yellow</material>
+</gazebo>
+<gazebo reference="pvc_up_left">
+  <material>Gazebo/Yellow</material>
+</gazebo>
+<gazebo reference="pvc_up_right">
+  <material>Gazebo/Yellow</material>
+</gazebo>
+<gazebo reference="pvc_45_left">
+  <material>Gazebo/Yellow</material>
+</gazebo>
+<gazebo reference="pvc_45_right">
+  <material>Gazebo/Yellow</material>
+</gazebo>
 </robot>
